File: ESP_NeoPixel.sch (EAGLE design)
At the start: 0 parts

Commit message: dimensions and wemos pins
Parts:
- added J1, J2: (no value), SparkFun-Connectors:CONN_08LOCK_NO_SILK
Connections:
- new net +3V3: J1.1
- new net +5V: J2.1
- new net A0: J1.7
- new net D0: J1.6
- new net D1: J2.6
- new net D2: J2.5
- new net D3: J2.4
- new net D4: J2.3
- new net D5: J1.5
- new net D6: J1.4
- new net D7: J1.3
- new net D8: J1.2
- new net GND: J2.2
- new net RST: J1.8
- new net RX: J2.7
- new net TX: J2.8
